Commit message: updates robot_config and getIK

File: i5_robots/i5_description/urdf/i5aubo1.xacro (robot description, xacro)
@@ -1,118 +1,84 @@
 <?xml version="1.0"?>
 <robot name="i5aubo1" xmlns:xacro="http://ros.org/wiki/xacro">
-    <!-- Constants -->
-    <xacro:property name="M_PI" value="3.14159"/>
+  <!-- Constants -->
+  <xacro:property name="M_PI" value="3.14159"/>
   <!-- ros_control plugin -->
-    <gazebo>
-        <plugin name="gazebo_ros_control" filename="libgazebo_ros_control.so">
-            <robotNamespace>/i5aubo1</robotNamespace>
-            <robotSimType>gazebo_ros_control/DefaultRobotHWSim</robotSimType>
-            <legacyModeNS>true</legacyModeNS>
-        </plugin>
-    </gazebo>
- <!-- Defining the colors used in this robot -->
-    <material name="Black">
-        <color rgba="0 0 0 1"/>
-    </material>
-    <material name="White">
+  <gazebo>
+    <plugin filename="libgazebo_ros_control.so" name="gazebo_ros_control">
+      <robotNamespace>/i5aubo1</robotNamespace>
+      <robotSimType>gazebo_ros_control/DefaultRobotHWSim</robotSimType>
+      <legacyModeNS>true</legacyModeNS>
+    </plugin>
+  </gazebo>
+  <!-- Defining the colors used in this robot -->
+  <material name="Black">
+    <color rgba="0 0 0 1"/>
+  </material>
+  <material name="White">
+    <color rgba="1 1 1 1"/>
+  </material>
+  <material name="Blue">
+    <color rgba="0 0 1 1"/>
+  </material>
+  <material name="Red">
+    <color rgba="1 0 0 1"/>
+  </material>
+  <material name="Grey">
+    <color rgba="0.96 0.96 0.96 1"/>
+  </material>
+  <!--/////////////////// DYNAMICS PARAM //////////////////////-->
+  <xacro:macro name="I5_Shoulder_Inertia">
+    <origin rpy="0 0 0" xyz="0.0 0.006 -0.002"/>
+    <mass value="5.05"/>
+    <inertia ixx="0.0148" ixy="0" ixz="0" iyy="0.0143" iyz="-0.0" izz="0.0095"/>
+  </xacro:macro>
+  <xacro:macro name="I5_UpperArm_Inertia">
+    <origin rpy="0 0 0" xyz="0.304 0.0 -0.03"/>
+    <mass value="11.90"/>
+    <inertia ixx="0.0305" ixy="0" ixz="0" iyy="0.4505" iyz="0" izz="0.0095"/>
+  </xacro:macro>
+  <xacro:macro name="I5_ForeArm_Inertia">
+    <origin rpy="0 0 0" xyz="0.415 0.0 0.0992"/>
+    <mass value="3.3"/>
+    <inertia ixx="0.0033" ixy="0" ixz="0.0009" iyy="0.0575" iyz="0" izz="0.0565"/>
+  </xacro:macro>
+  <xacro:macro name="I5_Wrist1_Inertia">
+    <origin rpy="0 0 0" xyz="0.0 0.0028 -0.003"/>
+    <mass value="1.62"/>
+    <inertia ixx="0.0023" ixy="0" ixz="0" iyy="0.0013" iyz="0.0" izz="0.0022"/>
+  </xacro:macro>
+  <xacro:macro name="I5_Wrist2_Inertia">
+    <origin rpy="0 0 0" xyz="0.0 -0.0028 -0.003"/>
+    <mass value="1.62"/>
+    <inertia ixx="0.0023" ixy="0" ixz="0" iyy="0.0013" iyz="0.0" izz="0.0022"/>
+  </xacro:macro>
+  <xacro:macro name="I5_Wrist3_Inertia">
+    <origin rpy="0 0 0" xyz="0.0 0.0 -0.0071"/>
+    <mass value="0.40"/>
+    <inertia ixx="0.013939" ixy="0" ixz="0" iyy="0.013988" iyz="0.0" izz="0.0224092"/>
+  </xacro:macro>
+  <!--/////////////////////////////// BASE_LINK ////////////////////////////////////-->
+  <link name="base_link">
+    <inertial>
+      <origin rpy="0 0 0" xyz="-1.4795E-13 0.0015384 0.020951"/>
+      <mass value="0.83419"/>
+      <inertia ixx="0.0014414" ixy="7.8809E-15" ixz="8.5328E-16" iyy="0.0013542" iyz="-1.4364E-05" izz="0.0024659"/>
+    </inertial>
+    <visual>
+      <origin rpy="0 0 0" xyz="0 0 0"/>
+      <geometry>
+         <!-- <mesh filename="package://aubo_description/meshes/aubo_i5/visual/base_link.DAE" /> -->
+         <mesh filename="package://i5_description/meshes/aubo_i5/visual/base_link.DAE" />
+        <!-- <mesh filename="$(arg description_directory)/meshes/aubo_i5/visual/base_link.DAE"/> -->
+      </geometry>
+      <material name="">
         <color rgba="1 1 1 1"/>
-    </material>
-    <material name="Blue">
-        <color rgba="0 0 1 1"/>
-    </material>
-    <material name="Red">
-        <color rgba="1 0 0 1"/>
-    </material>
-    <material name="Grey">
-        <color rgba="0.96 0.96 0.96 1"/>
-    </material>
-    <!--/////////////////// DYNAMICS PARAM //////////////////////-->
-    <xacro:macro name="I5_Shoulder_Inertia">
-        <origin xyz="0.0 0.006 -0.002"
-                rpy="0 0 0" />
-        <mass value="5.05" />
-        <inertia ixx="0.0148"
-                 ixy="0"
-                 ixz="0"
-                 iyy="0.0143"
-                 iyz="-0.0"
-                 izz="0.0095" />
-    </xacro:macro>
-    <xacro:macro name="I5_UpperArm_Inertia">
-        <origin xyz="0.304 0.0 -0.03"
-                rpy="0 0 0" />
-        <mass value="11.90" />
-        <inertia ixx="0.0305"
-                 ixy="0"
-                 ixz="0"
-                 iyy="0.4505"
-                 iyz="0"
-                 izz="0.0095" />
-    </xacro:macro>
-    <xacro:macro name="I5_ForeArm_Inertia">
-        <origin xyz="0.415 0.0 0.0992"
-                rpy="0 0 0" />
-        <mass  value="3.3" />
-        <inertia ixx="0.0033"
-                 ixy="0"
-                 ixz="0.0009"
-                 iyy="0.0575"
-                 iyz="0"
-                 izz="0.0565" />
-    </xacro:macro>
-    <xacro:macro name="I5_Wrist1_Inertia">
-        <origin xyz="0.0 0.0028 -0.003"
-                rpy="0 0 0" />
-        <mass value="1.62" />
-        <inertia ixx="0.0023"
-                 ixy="0"
-                 ixz="0"
-                 iyy="0.0013"
-                 iyz="0.0"
-                 izz="0.0022" />
-    </xacro:macro>
-    <xacro:macro name="I5_Wrist2_Inertia">
-        <origin xyz="0.0 -0.0028 -0.003"
-                rpy="0 0 0" />
-        <mass value="1.62" />
-        <inertia ixx="0.0023"
-                 ixy="0"
-                 ixz="0"
-                 iyy="0.0013"
-                 iyz="0.0"
-                 izz="0.0022" />
-    </xacro:macro>
-    <xacro:macro name="I5_Wrist3_Inertia">
-        <origin xyz="0.0 0.0 -0.0071"
-                rpy="0 0 0" />
-        <mass value="0.40" />
-        <inertia ixx="0.013939"
-                 ixy="0"
-                 ixz="0"
-                 iyy="0.013988"
-                 iyz="0.0"
-                 izz="0.0224092" />
-    </xacro:macro>
-    <!--/////////////////////////////// BASE_LINK ////////////////////////////////////-->
-   <link name="base_link">
-    <inertial>
-      <origin xyz="-1.4795E-13 0.0015384 0.020951" rpy="0 0 0" />
-      <mass value="0.83419" />
-      <inertia ixx="0.0014414" ixy="7.8809E-15" ixz="8.5328E-16" iyy="0.0013542" iyz="-1.4364E-05" izz="0.0024659" />
-    </inertial>
-    <visual>
-      <origin xyz="0 0 0" rpy="0 0 0" />
-      <geometry>
-        <!-- <mesh filename="package://aubo_description/meshes/aubo_i5/visual/base_link.DAE" /> -->
-        <mesh filename="/home/buivn/wsros_gazebo/src/i5_robots/i5_description/meshes/aubo_i5/visual/base_link.DAE" />
-      </geometry>
-      <material name="">
-        <color rgba="1 1 1 1" />
       </material>
     </visual>
     <collision>
-      <origin xyz="0 0 0" rpy="0 0 0" />
-      <geometry>
-        <mesh filename="/home/buivn/wsros_gazebo/src/i5_robots/i5_description/meshes/aubo_i5/collision/base_link.STL" />
+      <origin rpy="0 0 0" xyz="0 0 0"/>
+      <geometry>
+        <!-- <mesh filename="$(arg description_directory)/meshes/aubo_i5/collision/base_link.STL"/> -->
+        <mesh filename="package://i5_description/meshes/aubo_i5/collision/base_link.STL"/>
       </geometry>
     </collision>
@@ -121,19 +87,21 @@
   <link name="shoulder_Link">
     <inertial>
-      <xacro:I5_Shoulder_Inertia />
-    </inertial>
-    <visual>
-      <origin xyz="0 0 0" rpy="0 0 0" />
-      <geometry>
-        <mesh filename="/home/buivn/wsros_gazebo/src/i5_robots/i5_description/meshes/aubo_i5/visual/shoulder_Link.DAE" />
+      <xacro:I5_Shoulder_Inertia/>
+    </inertial>
+    <visual>
+      <origin rpy="0 0 0" xyz="0 0 0"/>
+      <geometry>
+        <!-- <mesh filename="$(arg description_directory)/meshes/aubo_i5/visual/shoulder_Link.DAE"/> -->
+        <mesh filename="package://i5_description/meshes/aubo_i5/visual/shoulder_Link.DAE"/>
       </geometry>
       <material name="">
-        <color rgba="1 1 1 1" />
+        <color rgba="1 1 1 1"/>
       </material>
     </visual>
     <collision>
-      <origin xyz="0 0 0" rpy="0 0 0" />
-      <geometry>
-        <mesh filename="/home/buivn/wsros_gazebo/src/i5_robots/i5_description/meshes/aubo_i5/collision/shoulder_Link.STL" />
+      <origin rpy="0 0 0" xyz="0 0 0"/>
+      <geometry>
+        <!-- <mesh filename="$(arg description_directory)/meshes/aubo_i5/collision/shoulder_Link.STL"/> -->
+        <mesh filename="package://i5_description/meshes/aubo_i5/collision/shoulder_Link.STL"/>
       </geometry>
     </collision>
@@ -141,28 +109,30 @@
   <!--/////////////////////////////// SHOULDER_JOINT ////////////////////////////////////-->
   <joint name="shoulder_joint" type="revolute">
-    <origin xyz="0 0 0.122" rpy="0 0 3.1416" />
-    <parent link="base_link" />
-    <child link="shoulder_Link" />
-    <axis xyz="0 0 1" />
-    <limit lower="-3.05" upper="3.05" effort="300" velocity="100" />
+    <origin rpy="0 0 3.1416" xyz="0 0 0.122"/>
+    <parent link="base_link"/>
+    <child link="shoulder_Link"/>
+    <axis xyz="0 0 1"/>
+    <limit effort="300" lower="-3.05" upper="3.05" velocity="100"/>
   </joint>
   <!--/////////////////////////////// UPPERARM_LINK ////////////////////////////////////-->
   <link name="upperArm_Link">
     <inertial>
-      <xacro:I5_UpperArm_Inertia />
-    </inertial>
-    <visual>
-      <origin xyz="0 0 0" rpy="0 0 0" />
-      <geometry>
-        <mesh filename="/home/buivn/wsros_gazebo/src/i5_robots/i5_description/meshes/aubo_i5/visual/upperArm_Link.DAE" />
+      <xacro:I5_UpperArm_Inertia/>
+    </inertial>
+    <visual>
+      <origin rpy="0 0 0" xyz="0 0 0"/>
+      <geometry>
+        <!-- <mesh filename="$(arg description_directory)/meshes/aubo_i5/visual/upperArm_Link.DAE"/> -->
+        <mesh filename="package://i5_description/meshes/aubo_i5/visual/upperArm_Link.DAE"/>
       </geometry>
       <material name="">
-        <color rgba="1 1 1 1" />
+        <color rgba="1 1 1 1"/>
       </material>
     </visual>
     <collision>
-      <origin xyz="0 0 0" rpy="0 0 0" />
-      <geometry>
-        <mesh filename="/home/buivn/wsros_gazebo/src/i5_robots/i5_description/meshes/aubo_i5/collision/upperArm_Link.STL" />
+      <origin rpy="0 0 0" xyz="0 0 0"/>
+      <geometry>
+        <!-- <mesh filename="$(arg description_directory)/meshes/aubo_i5/collision/upperArm_Link.STL"/> -->
+        <mesh filename="package://i5_description/meshes/aubo_i5/collision/upperArm_Link.STL"/>
       </geometry>
     </collision>
@@ -170,28 +140,30 @@
   <!--/////////////////////////////// UPPERARM_JOINT ////////////////////////////////////-->
   <joint name="upperArm_joint" type="revolute">
-    <origin xyz="0 0.1215 0" rpy="-1.5708 -1.5708 0" />
-    <parent link="shoulder_Link" />
-    <child link="upperArm_Link" />
-    <axis xyz="0 0 1" />
-    <limit lower="-3.05" upper="3.05" effort="300" velocity="100" />
+    <origin rpy="-1.5708 -1.5708 0" xyz="0 0.1215 0"/>
+    <parent link="shoulder_Link"/>
+    <child link="upperArm_Link"/>
+    <axis xyz="0 0 1"/>
+    <limit effort="300" lower="-3.05" upper="3.05" velocity="100"/>
   </joint>
   <!--/////////////////////////////// FOREARM_LINK ////////////////////////////////////-->
   <link name="foreArm_Link">
     <inertial>
-      <xacro:I5_ForeArm_Inertia />
-    </inertial>
-    <visual>
-      <origin xyz="0 0 0" rpy="0 0 0" />
-      <geometry>
-        <mesh filename="/home/buivn/wsros_gazebo/src/i5_robots/i5_description/meshes/aubo_i5/visual/foreArm_Link.DAE" />
+      <xacro:I5_ForeArm_Inertia/>
+    </inertial>
+    <visual>
+      <origin rpy="0 0 0" xyz="0 0 0"/>
+      <geometry>
+        <!-- <mesh filename="$(arg description_directory)/meshes/aubo_i5/visual/foreArm_Link.DAE"/> -->
+        <mesh filename="package://i5_description/meshes/aubo_i5/visual/foreArm_Link.DAE"/>
       </geometry>
       <material name="">
-        <color rgba="1 1 1 1" />
+        <color rgba="1 1 1 1"/>
       </material>
     </visual>
     <collision>
-      <origin xyz="0 0 0" rpy="0 0 0" />
-      <geometry>
-        <mesh filename="/home/buivn/wsros_gazebo/src/i5_robots/i5_description/meshes/aubo_i5/collision/foreArm_Link.STL" />
+      <origin rpy="0 0 0" xyz="0 0 0"/>
+      <geometry>
+        <!-- <mesh filename="$(arg description_directory)/meshes/aubo_i5/collision/foreArm_Link.STL"/> -->
+        <mesh filename="package://i5_description/meshes/aubo_i5/collision/foreArm_Link.STL"/>
       </geometry>
     </collision>
@@ -199,28 +171,30 @@
   <!--/////////////////////////////// FOREARM_JOINT ////////////////////////////////////-->
   <joint name="foreArm_joint" type="revolute">
-    <origin xyz="0.408 0 0" rpy="-3.1416 -5.1632E-18 -5.459E-16" />
-    <parent link="upperArm_Link" />
-    <child link="foreArm_Link" />
-    <axis xyz="0 0 1" />
-    <limit lower="-3.05" upper="3.05" effort="300" velocity="100" />
+    <origin rpy="-3.1416 -5.1632E-18 -5.459E-16" xyz="0.408 0 0"/>
+    <parent link="upperArm_Link"/>
+    <child link="foreArm_Link"/>
+    <axis xyz="0 0 1"/>
+    <limit effort="300" lower="-3.05" upper="3.05" velocity="100"/>
   </joint>
   <!--/////////////////////////////// WRIST1_LINK ////////////////////////////////////-->
   <link name="wrist1_Link">
     <inertial>
-      <xacro:I5_Wrist1_Inertia />
-    </inertial>
-    <visual>
-      <origin xyz="0 0 0" rpy="0 0 0" />
-      <geometry>
-        <mesh filename="/home/buivn/wsros_gazebo/src/i5_robots/i5_description/meshes/aubo_i5/visual/wrist1_Link.DAE" />
+      <xacro:I5_Wrist1_Inertia/>
+    </inertial>
+    <visual>
+      <origin rpy="0 0 0" xyz="0 0 0"/>
+      <geometry>
+        <!-- <mesh filename="$(arg description_directory)/meshes/aubo_i5/visual/wrist1_Link.DAE"/> -->
+        <mesh filename="package://i5_description/meshes/aubo_i5/visual/wrist1_Link.DAE"/>
       </geometry>
       <material name="">
-        <color rgba="1 1 1 1" />
+        <color rgba="1 1 1 1"/>
       </material>
     </visual>
     <collision>
-      <origin xyz="0 0 0" rpy="0 0 0" />
-      <geometry>
-        <mesh filename="/home/buivn/wsros_gazebo/src/i5_robots/i5_description/meshes/aubo_i5/collision/wrist1_Link.STL" />
+      <origin rpy="0 0 0" xyz="0 0 0"/>
+      <geometry>
+        <!-- <mesh filename="$(arg description_directory)/meshes/aubo_i5/collision/wrist1_Link.STL"/> -->
+        <mesh filename="package://i5_description/meshes/aubo_i5/collision/wrist1_Link.STL"/>
       </geometry>
     </collision>
@@ -228,28 +202,30 @@
   <!--/////////////////////////////// WRIST1_JOINT ////////////////////////////////////-->
   <joint name="wrist1_joint" type="revolute">
-    <origin xyz="0.376 0 0" rpy="3.1416 -1.8323E-15 1.5708" />
-    <parent link="foreArm_Link" />
-    <child link="wrist1_Link" />
-    <axis xyz="0 0 1" />
-    <limit lower="-3.05" upper="3.05" effort="300" velocity="100" />
+    <origin rpy="3.1416 -1.8323E-15 1.5708" xyz="0.376 0 0"/>
+    <parent link="foreArm_Link"/>
+    <child link="wrist1_Link"/>
+    <axis xyz="0 0 1"/>
+    <limit effort="300" lower="-3.05" upper="3.05" velocity="100"/>
   </joint>
   <!--/////////////////////////////// WRIST2_LINK ////////////////////////////////////-->
   <link name="wrist2_Link">
     <inertial>
-      <xacro:I5_Wrist2_Inertia />
-    </inertial>
-    <visual>
-      <origin xyz="0 0 0" rpy="0 0 0" />
-      <geometry>
-        <mesh filename="/home/buivn/wsros_gazebo/src/i5_robots/i5_description/meshes/aubo_i5/visual/wrist2_Link.DAE" />
+      <xacro:I5_Wrist2_Inertia/>
+    </inertial>
+    <visual>
+      <origin rpy="0 0 0" xyz="0 0 0"/>
+      <geometry>
+        <!-- <mesh filename="$(arg description_directory)/meshes/aubo_i5/visual/wrist2_Link.DAE"/> -->
+        <mesh filename="package://i5_description/meshes/aubo_i5/visual/wrist2_Link.DAE"/>
       </geometry>
       <material name="">
-        <color rgba="1 1 1 1" />
+        <color rgba="1 1 1 1"/>
       </material>
     </visual>
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